Commit message: changes for local building

File: ur_moveit_config/srdf/ur.srdf.xacro (robot description, xacro)
@@ -3,5 +3,5 @@
   <!-- robot name parameter -->
   <xacro:arg name="name" default="ur"/>
-  <xacro:include filename="$(find ur_moveit_config)/srdf/ur_macro.srdf.xacro"/>
+  <xacro:include filename="$(find ur_moveit_config)/srdf/ur_bam_macro.srdf.xacro"/>
   <xacro:ur_srdf/>
 </robot>

File: ur_moveit_config/srdf/ur_bam_macro.srdf.xacro (robot description, xacro)
@@ -53,4 +53,16 @@
     <disable_collisions link1="wrist_1_link" link2="wrist_3_link" reason="Never" />
     <disable_collisions link1="wrist_2_link" link2="wrist_3_link" reason="Adjacent" />
+    <group name="eef">
+        <link name="eef_link_1"/>
+        <link name="eef_link_2"/>
+    </group>
+    <!--END EFFECTOR: Purpose: Represent information about an end effector.-->
+    <end_effector name="eef" parent_link="tool0" group="eef" parent_group="ur_manipulator"/>
+    <!--PASSIVE JOINT: Purpose: this element is used to mark joints that are not actuated-->
+    <!-- <passive_joint name="joint_virtual_finger"/> -->
+    <disable_collisions link1="eef_link_1" link2="eef_link_2" reason="Adjacent"/>
+    <disable_collisions link1="eef_link_1" link2="wrist_2_link" reason="Adjacent"/>
+    <disable_collisions link1="eef_link_1" link2="wrist_3_link" reason="Adjacent"/>
+    <disable_collisions link1="eef_link_2" link2="wrist_3_link" reason="Adjacent"/>
   </xacro:macro>
 </robot>

Commit message: adding ur baseline to core.launch.py for plugin:=mock and gripper:=none,crab_claw

File: ur_moveit_config/srdf/ur.srdf.xacro (robot description, xacro)
@@ -3,6 +3,7 @@
   <!-- robot name parameter -->
   <xacro:arg name="name" default="ur"/>
-  <!-- <xacro:include filename="$(find ur_moveit_config)/srdf/ur_bam_macro.srdf.xacro"/> -->
-  <xacro:include filename="$(find ur_moveit_config)/srdf/ur_macro.srdf.xacro"/>
-  <xacro:ur_srdf/>
+  <xacro:arg name="gripper" default="none"/>
+  <xacro:include filename="$(find ur_moveit_config)/srdf/ur_bam_macro.srdf.xacro"/>
+  <!-- <xacro:include filename="$(find ur_moveit_config)/srdf/ur_macro.srdf.xacro"/> -->
+  <xacro:ur_srdf gripper="$(arg gripper)"/>
 </robot>

File: ur_moveit_config/srdf/ur_bam_macro.srdf.xacro (robot description, xacro)
@@ -5,5 +5,5 @@
     A URDF file must exist for this robot as well, where the joints and the links that are referenced are defined
 -->
-  <xacro:macro name="ur_srdf" params="">
+  <xacro:macro name="ur_srdf" params="gripper">
     <!--GROUPS - Representation of a set of joints and links. This can be useful for specifying DOF to plan for, defining arms, end effectors, etc-->
     <!--LINKS - When a link is specified, the parent joint of that link (if it exists) is automatically included-->
@@ -53,16 +53,18 @@
     <disable_collisions link1="wrist_1_link" link2="wrist_3_link" reason="Never" />
     <disable_collisions link1="wrist_2_link" link2="wrist_3_link" reason="Adjacent" />
-    <group name="eef">
-        <link name="eef_link_1"/>
-        <link name="eef_link_2"/>
-    </group>
-    <!--END EFFECTOR: Purpose: Represent information about an end effector.-->
-    <end_effector name="eef" parent_link="tool0" group="eef" parent_group="ur_manipulator"/>
-    <!--PASSIVE JOINT: Purpose: this element is used to mark joints that are not actuated-->
-    <!-- <passive_joint name="joint_virtual_finger"/> -->
-    <disable_collisions link1="eef_link_1" link2="eef_link_2" reason="Adjacent"/>
-    <disable_collisions link1="eef_link_1" link2="wrist_2_link" reason="Adjacent"/>
-    <disable_collisions link1="eef_link_1" link2="wrist_3_link" reason="Adjacent"/>
-    <disable_collisions link1="eef_link_2" link2="wrist_3_link" reason="Adjacent"/>
+    <xacro:if value="${gripper != 'none'}">
+      <group name="eef">
+          <link name="eef_link_1"/>
+          <link name="eef_link_2"/>
+      </group>
+      <!--END EFFECTOR: Purpose: Represent information about an end effector.-->
+      <end_effector name="eef" parent_link="ee_link" group="eef" parent_group="ur_manipulator"/>
+      <!--PASSIVE JOINT: Purpose: this element is used to mark joints that are not actuated-->
+      <!-- <passive_joint name="joint_virtual_finger"/> -->
+      <disable_collisions link1="eef_link_1" link2="eef_link_2" reason="Adjacent"/>
+      <disable_collisions link1="eef_link_1" link2="wrist_2_link" reason="Adjacent"/>
+      <disable_collisions link1="eef_link_1" link2="wrist_3_link" reason="Adjacent"/>
+      <disable_collisions link1="eef_link_2" link2="wrist_3_link" reason="Adjacent"/>
+    </xacro:if>
   </xacro:macro>
 </robot>
